File: schematic/schematic.kicad_sch (KiCad schematic)
At the start: 13 parts, among them J1 Screw_Terminal_01x10, K1 External relay for pressure s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, K3 External relay for dust sensor, U1 ESP32-WROOM-32, U2 DS18B20

Commit message: Update schematic.
Parts:
- removed J1: Screw_Terminal_01x10, symbol Connector:Screw_Terminal_01x10
- removed K1: External relay for pressure sensor, Relay_THT:Relay_SPST-NO_Fujitsu_FTR-LYAA005x_FormA_Vertical, symbol Relay:Fujitsu_FTR-LYAA005x
- removed K3: External relay for dust sensor, Relay_THT:Relay_SPST-NO_Fujitsu_FTR-LYAA005x_FormA_Vertical, symbol Relay:Fujitsu_FTR-LYAA005x
- removed R5: 1k, symbol Device:R
- removed RV1: Ultrasonic dust sensor, symbol Device:R_Potentiometer
- added D1, D4: RED 24V, symbol Device:LED
- added D2: YELLOW 24V, symbol Device:LED
- added D3: GREEN 24V, symbol Device:LED
- added J1: Screw_Terminal_01x16, symbol Connector:Screw_Terminal_01x16
- added J2, J6: Screw_Terminal_01x06, symbol Connector:Screw_Terminal_01x06
- added K2: External relay for dust collector motor, Relay_THT:Relay_SPST-NO_Fujitsu_FTR-LYAA005x_FormA_Vertical, symbol Relay:Fujitsu_FTR-LYAA005x
- added K5: Pressure sensor relay, Relay_THT:Relay_SPDT_Fujitsu_FTR-LYCA005x_FormC_Vertical, symbol Relay:Fujitsu_FTR-LYCA005x
- added M1: Dust collector motor, symbol Motor:Motor_AC
- added M2: 16-channel multiplexer, symbol Symbols:Multiplexer16
- added Q1: IRF520N, Package_TO_SOT_THT:TO-220-3_Vertical, symbol Transistor_FET:IRF540N
- added R11, R12, R13, R14: 1.5k, symbol Device:R
- added R7: 10K, symbol Device:R
- added R8, R9: 10k, symbol Device:R
- added U4: Ultrasonic range sensor, symbol Symbols:UltrasonicRangeSensor
- added U5: Scale Module, symbol Symbols:ScaleModule
- C1: value 200-400uF -> 200-500uF
- R1: value 4.7k -> 10k
- R2: value 1k -> 120 Ohm
- R3: value 3k -> 4.7k
- R4: value 1k -> 10k
- U2, U3: now left out of the parts list
Connections:
- net GND: now also D1.1 (K), D2.1 (K), D3.1 (K), D4.1 (K), J2.1 (Pin_1), J6.1 (Pin_1), J6.2 (Pin_2), J6.3 (Pin_3), J6.4 (Pin_4), J6.5 (Pin_5), J6.6 (Pin_6), M1.1, M2. (GND), Q1.3 (S), R11.2, R12.2, R13.2, R14.2, R7.2, U4. (Output), U5.17 (DC24V(-))
- net Onewire bus: now also R3.1, J2.5 (Pin_5); no longer R1.2
- net 5V: now reaches C1.1, U1.40 (5V_IN), U3. (GND)
- net 5V: now also J2.3 (Pin_3)
- net 3.3V: now reaches U1.2 (3.3V), U2.3 (V_{DD})
- net 3.3V: now also R3.2, J2.2 (Pin_2), M2. (GND); no longer R1.1
- net at R4.1: now also M2. (GND), R14.1
- net at U1.12 (IO27): now also Q1.1 (G), R7.1
- net S0: now reaches U1.14 (IO12)
- net S0: now also M2. (GND)
- net S3: now reaches U1.25 (IO0)
- net S3: now also M2. (GND)
- net S2: now reaches U1.26 (IO4)
- net S2: now also M2. (GND)
- net SIG: now reaches U1.33 (IO21)
- net SIG: now also M2. (GND)
- removed net Dust sensor: R2.2, R3.1, U1.27 (IO16)
- net Dust sensor switch renamed Dust sensor loop 2
- net Dust sensor loop 2: now also R2.2, J2.6 (Pin_6), U5.14 (Sensor_COM)
- net Pressure sensor switch: no longer names the net of U1.16 (IO13)
- net Pressure sensor switch: no longer R4.2
- new net: K2.14, M1.2
- new net: M2. (GND), R13.1, R8.1
- new net: M2. (GND), R11.1, R9.1
- new net: K5.14, U5.24 (COM)
- new net: M2. (GND), R1.1, R12.1
- new net 24V: J2.4 (Pin_4), K5.11, U3. (GND), U4. (Output)
- new net Dust sensor loop 1: U4. (Output), U5.15 (Sensor_Current)
- new net Dust warning signal 1: D2.2 (A), J1.14 (Pin_14), R1.2, U5.20 (AL3)
- new net Dust warning signal 2: D1.2 (A), J1.15 (Pin_15), R8.2, U5.19 (AL2)
- new net Gate 1: J1.1 (Pin_1), M2. (GND)
- new net Gate 10: J1.10 (Pin_10), M2. (GND)
- new net Gate 11: J1.11 (Pin_11), M2. (GND)
- new net Gate 12: J1.12 (Pin_12), M2. (GND)
- new net Gate 2: J1.2 (Pin_2), M2. (GND)
- new net Gate 3: J1.3 (Pin_3), M2. (GND)
- new net Gate 4: J1.4 (Pin_4), M2. (GND)
- new net Gate 5: J1.5 (Pin_5), M2. (GND)
- new net Gate 6: J1.6 (Pin_6), M2. (GND)
- new net Gate 7: J1.7 (Pin_7), M2. (GND)
- new net Gate 8: J1.8 (Pin_8), M2. (GND)
- new net Gate 9: J1.9 (Pin_9), M2. (GND)
- new net Low pressure signal: D4.2 (A), J1.13 (Pin_13), K5.12, R9.2
- new net Main power relay: D3.2 (A)
- new net Main power relay (+): K2.A2, U5.18 (AL1)
- new net Main power relay (-): J1.16 (Pin_16), K2.A1, Q1.2 (D), R4.2
- new net S1: M2. (GND), U1.27 (IO16)
- new net Three phase AC: K2.13
- no-connect marks 0 -> 3
Other:
- note added: "(4-20 mA)"
- note added: "5V PSU"
- note added: "Also serves as pull-downs"
- note added: "Current sensing"
- note added: "ESP32 Controller board"
- note added: "ESP32 code & schematic source"
- note added: "Flashing warning light"
- note added: "Indicator light tower"
- note added: "Main power relay"
- note added: "Main power relay (+) = 24V (on) / Floating (off) - High side controlled by sensor relays Main power relay (-) = GND (on) / Floating (off) - Low side controlled by MCU Dust warning signal 1 = 24V (warning) / Floating (no warning) - When dust bin should be emptied, but machine can still run Dust warning signal 2 = 24V (warning) / Floating (no warning) - When dust bin should be emptied, and machine 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"
- note added: "Not really how the connections look, but I didn't find a good three phase relay and motor symbol"
- note added: "ON = Dust < ~90%"
- note added: "ON = Dust > ~80%"
- note added: "ON = Dust > ~90%"
- note added: "Pressure sensor"
- note added: "Pulldown (works even if MCU is unpowered)"
- note added: "Scale module"
- note added: "Temperature sensor"
- note added: "Ultrasonic dust sensor"
- note added: "Voltage dividers 24V->~3.3V"
- note removed: "Protection resistors for transients"
- note removed: "Voltage divider 10V->2.5V"
- company: (none) -> Stockholm Makerspace
- title: (none) -> Dust Collector Controller
- moved on the sheet: C1, R2, U1, U2, U3

Commit message: Update schematic.
Parts:
- removed J2, J6: Screw_Terminal_01x06, symbol Connector:Screw_Terminal_01x06
- removed R11, R12, R13, R14: 1.5k, symbol Device:R
- removed R8, R9: 10k, symbol Device:R
- added J2: Screw_Terminal_01x07, symbol Connector:Screw_Terminal_01x07
- added J3: Screw_Terminal_01x10, symbol Connector:Screw_Terminal_01x10
- added R5, R6: 3k, symbol Device:R
- added U6, U7, U8, U9: Optocoupler_DC_PhotoNPN_AKEC, symbol Isolator:Optocoupler_DC_PhotoNPN_AKEC
- R1, R4: value 10k -> 3k
Connections:
- net 24V: now also J2.4 (Pin_4)
- net 3.3V: now also J2.2 (Pin_2)
- net 5V: now also J2.3 (Pin_3)
- net Dust sensor loop 2: now also J2.6 (Pin_6)
- net Dust warning signal 1: now also R4.1; no longer J1.14 (Pin_14), R1.2
- net Dust warning signal 2: now also R5.1; no longer J1.15 (Pin_15)
- net GND: now also J2.1 (Pin_1), J3.1 (Pin_1), J3.10 (Pin_10), J3.2 (Pin_2), J3.3 (Pin_3), J3.4 (Pin_4), J3.5 (Pin_5), J3.6 (Pin_6), J3.7 (Pin_7), J3.8 (Pin_8), J3.9 (Pin_9), U6.2, U6.3, U7.2, U7.3, U8.2, U8.3, U9.2, U9.3
- net Low pressure signal: now also R1.1; no longer J1.13 (Pin_13)
- net Main power relay (-): now also J2.7 (Pin_7), R6.1; no longer J1.16 (Pin_16), R4.2
- net Onewire bus: now also J2.5 (Pin_5)
- new net: R4.2, U7.1
- new net: R6.2, U9.1
- new net: R5.2, U8.1
- new net: R1.2, U6.1
- new net Dust warning signal 1 (LV): J1.14 (Pin_14), M2. (GND), U7.4
- new net Dust warning signal 2 (LV): J1.15 (Pin_15), M2. (GND), U8.4
- new net Low pressure signal (LV): J1.13 (Pin_13), M2. (GND), U6.4
- new net Main power relay (-, LV): J1.16 (Pin_16), M2. (GND), U9.4
Other:
- note added: "Optocoupler Module"
- note added: "To gates and optocoupler"
- note removed: "Also serves as pull-downs"
- note removed: "Voltage dividers 24V->~3.3V"
- moved on the sheet: J1, Q1, R2, R3, R7

Commit message: Update schematic.
Parts:
- added J4: Screw_Terminal_01x02, symbol Connector:Screw_Terminal_01x02
- added V1: 24V, symbol Simulation_SPICE:VDC
- R7: value 10K -> 12k
Connections:
- net Main power relay is gone; now on net Main power relay (+): D3.2 (A)
- net 24V: now also U3.1 (24V), V1.1; no longer U3. (GND)
- net 3.3V: now also R3.1; no longer R3.2
- net 5V: now also U3.2 (5V); no longer U3. (GND)
- net Dust sensor loop 2: now also U1.16 (IO13); no longer U1.13 (IO14)
- net Dust warning signal 1 (LV): now also J1.2 (Pin_2); no longer J1.14 (Pin_14)
- net Dust warning signal 2 (LV): now also J1.3 (Pin_3); no longer J1.15 (Pin_15)
- net GND: now also U3.3 (GND), U3.4 (GND), J4.1 (Pin_1), J4.2 (Pin_2), V1.2; no longer U3. (GND)
- net Gate 1: now also J1.5 (Pin_5); no longer J1.1 (Pin_1)
- net Gate 10: now also J1.14 (Pin_14); no longer J1.10 (Pin_10)
- net Gate 11: now also J1.15 (Pin_15); no longer J1.11 (Pin_11)
- net Gate 12: now also J1.16 (Pin_16); no longer J1.12 (Pin_12)
- net Gate 2: now also J1.6 (Pin_6); no longer J1.2 (Pin_2)
- net Gate 3: now also J1.7 (Pin_7); no longer J1.3 (Pin_3)
- net Gate 4: now also J1.8 (Pin_8); no longer J1.4 (Pin_4)
- net Gate 5: now also J1.9 (Pin_9); no longer J1.5 (Pin_5)
- net Gate 6: now also J1.10 (Pin_10); no longer J1.6 (Pin_6)
- net Gate 7: now also J1.11 (Pin_11); no longer J1.7 (Pin_7)
- net Gate 8: now also J1.12 (Pin_12); no longer J1.8 (Pin_8)
- net Gate 9: now also J1.13 (Pin_13); no longer J1.9 (Pin_9)
- net Low pressure signal (LV): now also J1.1 (Pin_1); no longer J1.13 (Pin_13)
- net Main power relay (-, LV): now also J1.4 (Pin_4); no longer J1.16 (Pin_16)
- net Onewire bus: now also R3.2, U1.37 (IO23); no longer R3.1, U1.23 (IO15)
- net S0: now also U1.13 (IO14); no longer U1.14 (IO12)
- net S1: now also U1.12 (IO27); no longer U1.27 (IO16)
- net S2: now also U1.11 (IO26); no longer U1.26 (IO4)
- net S3: now also U1.10 (IO25); no longer U1.25 (IO0)
- net SIG: now also U1.9 (IO33); no longer U1.33 (IO21)
- net High pressure signal: now reaches K5.14, U5.24 (COM)
- net Main power control: now reaches Q1.1 (G), R7.1
- net Main power control: now also U1.14 (IO12); no longer U1.12 (IO27)
- no-connect marks 3 -> 29
Other:
- note added: "24V PSU"
- note added: "Pulldown (for unpowered MCU)"
- note removed: "5V PSU"
- note removed: "Pulldown (works even if MCU is unpowered)"
- moved on the sheet: C1, J1, J2, J3, K2, K5, M1, M2, Q1, R2, R3, R7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
