File: schematic2/ESP32-devboard.kicad_sch (KiCad schematic)
At the start: 104 parts, among them J1 CON19x1-LEFT, J10 Screw_Terminal_01x12, J2 CON19x1-RIGHT, J3 GT-USB-7010ASV, J4 Screw_Terminal_01x10, J5 Screw_Terminal_01x07, J6 Screw_Terminal_01x02, J7 Screw_Terminal_01x10, J8 Screw_Terminal_01x16, K1 Pressure sensor relay, K2 External relay for dust colle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, M1 Dust collector motor, Q1 SS8050 200-350, Q2 HL3400, Q3 SS8050 200-350, Q4 HL3400, Q5 HL3400, Q6 IRF520N, U1 ESP32-WROOM-E, U10 Ultrasonic range sensor, U11 DS18B20, U12 Scale Module, U13 LTV-217-B-G, U14 LTV-217-B-G, U15 LTV-217-B-G, U16 LTV-217-B-G, U2 CP2102N-Axx-xQFN28, U3 AMS1117-3.3, U4 XL1509, U5 CD4051BM96, U6 Optocoupler_DC_PhotoNPN_AKEC, U7 Optocoupler_DC_PhotoNPN_AKEC, U8 Optocoupler_DC_PhotoNPN_AKEC, U9 Optocoupler_DC_PhotoNPN_AKEC

Commit message: Schematic updates
Parts:
- removed R38: 1k(5%), Capacitor_SMD:C_0603_1608Metric, symbol Device:R
- added D18, D19, D20, D21, D22, D23, D24, D25, D26, D27, D28, D29: Green, PCM_JLCPCB:D_0805, symbol PCM_JLCPCB-Diodes:LED,0805,Green
- added J9: Screw_Terminal_01x04, TerminalBlock_Phoenix:TerminalBlock_Phoenix_MKDS-1,5-4_1x04_P5.00mm_Horizontal, symbol Connector:Screw_Terminal_01x04
- added R29, R34, R35, R36, R43, R44, R45, R46, R51, R52, R53, R54, R55: 2k(5%), Capacitor_SMD:C_0603_1608Metric, symbol Device:R
- added R30, R31, R32, R33, R39, R40, R41, R42, R47, R48, R49, R50: 20K(5%), Capacitor_SMD:C_0603_1608Metric, symbol Device:R
- added U17, U18, U19, U20, U21, U22, U23, U24, U25, U26, U27, U28: LTV-217-B-G, PCM_JLCPCB:SOP-4_4.4x2.6mm_P1.27mm, symbol PCM_JLCPCB-Optocouplers:LTV-217-B-G
- added U29: CD4051BM96, PCM_JLCPCB:SOIC-16_L9.9-W3.9-P1.27-LS6.0-BL, symbol PCM_JLCPCB-Analog:Switch, CD4051BM96
- R18, R25, R37: value 10K(5%) -> 20K(5%)
- R24, R28: value 1k(5%) -> 2k(5%)
- R26: value 1k(5%) -> 20K(5%)
- R27: value 10K(5%) -> 2k(5%)
Connections:
- net 3.3V: now also U17.4, U18.4, U19.4, U20.4, U21.4, U22.4, U23.4, U24.4, U25.4, U26.4, U27.4, U28.4, U29.16 (VDD)
- net GND: now also R24.2, R26.1, R27.2, R28.2, R29.2, R30.1, R31.1, R32.1, R33.1, R34.2, R35.2, R36.2, R39.1, R40.1, R41.1, R42.1, R43.2, R44.2, R45.2, R46.2, R47.1, R48.1, R49.1, R50.1, R51.2, R52.2, R53.2, R54.2, R55.2, U29.6 (INH), U29.7 (VEE), U29.8 (VSS); no longer D14.1, D15.1, D16.1, D17.1, R27.1, U13.2, U14.2, U15.2, U16.2
- net Gate 1: now also U29.12 (CHANNELS_IN/OUT_3); no longer R18.2, R24.2, R25.2, R26.2, R27.2, R28.2, U13.3, U15.3, U16.3, U5.13 (CHANNELS_IN/OUT_0)
- net Gate 2: now also R18.2, U13.3, U29.13 (CHANNELS_IN/OUT_0); no longer U5.14 (CHANNELS_IN/OUT_1)
- net Gate 3: now also R25.2, U15.3, U29.14 (CHANNELS_IN/OUT_1); no longer U5.15 (CHANNELS_IN/OUT_2)
- net Gate 4: now also R26.2, U16.3, U29.15 (CHANNELS_IN/OUT_2); no longer U5.12 (CHANNELS_IN/OUT_3)
- net Gate 5: now also U5.5 (IN/OUT_5), R30.2, U17.3; no longer U5.1 (CHANNELS_4)
- net Gate 6: now also U5.4 (CHANNELS_7), R31.2, U18.3; no longer U5.5 (IN/OUT_5)
- net Gate 7: now also R32.2, U19.3
- net Gate 8: now also U5.1 (CHANNELS_4), R33.2, U20.3; no longer U5.4 (CHANNELS_7)
- net IO25: now also U29.9 (C)
- net IO26: now also U29.10 (B)
- net IO27: now also U29.11 (A)
- net IO33: now also U29.3 (COM_OUT/IN)
- net at R28.1: now also D17.1; no longer D17.2
- net at J10.10 (Pin_10): now also U22.1
- net at J10.11 (Pin_11): now also U23.1
- net at J10.12 (Pin_12): now also U24.1
- net at J10.5 (Pin_5): now also U17.1
- net at J10.6 (Pin_6): now also U18.1
- net at J10.7 (Pin_7): now also U19.1
- net at J10.8 (Pin_8): now also U20.1
- net at J10.9 (Pin_9): now also U21.1
- net at D14.2: now also U14.2
- net at D16.2: now also U15.2; no longer R26.1
- net at D15.2: now also U13.2; no longer R24.1
- new net: D28.1, R53.1
- new net: D28.2, U27.2
- new net: D17.2, U16.2
- new net: D18.1, R34.1
- new net: J9.4 (Pin_4), U28.1
- new net: D29.2, U28.2
- new net: D22.2, U21.2
- new net: D26.1, R51.1
- new net: D14.1, R29.1
- new net: D21.1, R55.1
- new net: D21.2, U20.2
- new net: D23.1, R44.1
- new net: D19.1, R35.1
- new net: D19.2, U18.2
- new net: D27.1, R52.1
- new net: D27.2, U26.2
- new net: D25.2, U24.2
- new net: D25.1, R46.1
- new net: D22.1, R43.1
- new net: D23.2, U22.2
- new net: D16.1, R27.1
- new net: D20.2, U19.2
- new net: D24.1, R45.1
- new net: D24.2, U23.2
- new net: J9.1 (Pin_1), U25.1
- new net: D26.2, U25.2
- new net: J9.3 (Pin_3), U27.1
- new net: D18.2, U17.2
- new net: D20.1, R36.1
- new net: D15.1, R24.1
- new net: D29.1, R54.1
- new net: J9.2 (Pin_2), U26.1
- new net Gate 10: R40.2, U22.3, U5.13 (CHANNELS_IN/OUT_0)
- new net Gate 11: R41.2, U23.3, U5.14 (CHANNELS_IN/OUT_1)
- new net Gate 12: R42.2, U24.3, U5.15 (CHANNELS_IN/OUT_2)
- new net Gate 9: R39.2, U21.3, U5.12 (CHANNELS_IN/OUT_3)
- new net Gate B1: R47.2, U25.3, U29.5 (IN/OUT_5)
- new net Gate B2: R48.2, U26.3, U29.4 (CHANNELS_7)
- new net Gate B3: R49.2, U27.3, U29.2 (IN/OUT_6)
- new net Gate B4: R50.2, U28.3, U29.1 (CHANNELS_4)
Other:
- moved on the sheet: D10, D11, D12, D13, D14, J10, R37, U14, U5

Commit message: Schematic updates - Ordered from JLCPCB
Parts:
- removed D13: RED 24V, symbol Device:LED
- removed D5: Red, PCM_JLCPCB:D_0603, symbol PCM_JLCPCB-Diodes:LED,0603,Red
- removed J5: Screw_Terminal_01x07, symbol Connector:Screw_Terminal_01x07
- removed J6: Screw_Terminal_01x02, symbol Connector:Screw_Terminal_01x02
- removed J7: Screw_Terminal_01x10, symbol Connector:Screw_Terminal_01x10
- removed J8: Screw_Terminal_01x16, TerminalBlock_Phoenix:TerminalBlock_Phoenix_MKDS-1,5-16_1x16_P5.00mm_Horizontal, symbol Connector:Screw_Terminal_01x16
- removed JP1: Jumper_2_Bridged, Connector_PinHeader_2.54mm:PinHeader_1x02_P2.54mm_Vertical, symbol Jumper:Jumper_2_Bridged
- removed Q6: IRF520N, Package_TO_SOT_THT:TO-220-3_Vertical, symbol Transistor_FET:IRF540N
- removed R23: 2K(5%), Capacitor_SMD:C_0603_1608Metric, symbol Device:R
- removed RV1: 10k, Potentiometer_SMD:Potentiometer_Bourns_TC33X_Vertical, symbol Device:R_Potentiometer
- removed U12: Scale Module, symbol Symbols:ScaleModule
- removed U6, U7, U8, U9: Optocoupler_DC_PhotoNPN_AKEC, symbol Isolator:Optocoupler_DC_PhotoNPN_AKEC
- added BZ1: Buzzer, symbol Device:Buzzer
- added C13, C14: 0.1uF/50V(10%), Capacitor_SMD:C_0402_1005Metric, symbol Device:C
- added D13, D30: Green, PCM_JLCPCB:D_0805, symbol PCM_JLCPCB-Diodes:LED,0805,Green
- added D32: Red, PCM_JLCPCB:D_0603, symbol PCM_JLCPCB-Diodes:LED,0603,Red
- added D33, D5: Yellow, PCM_JLCPCB:D_0805, symbol PCM_JLCPCB-Diodes:LED,0805,Yellow
- added J11, J5, J6, J8: Screw_Terminal_01x03, Connector_PinHeader_2.54mm:PinHeader_1x03_P2.54mm_Horizontal, symbol Connector:Screw_Terminal_01x03
- added J7: Screw_Terminal_01x08, TerminalBlock_Phoenix:TerminalBlock_Phoenix_MKDS-1,5-8_1x08_P5.00mm_Horizontal, symbol Connector:Screw_Terminal_01x08
- added Q10, Q11, Q13, Q7: MMBT3904 100-300, PCM_JLCPCB:Q_SOT-23, symbol PCM_JLCPCB-Transistors:NPN,MMBT3904 100-300
- added Q12, Q14, Q8, Q9: AO3401A, PCM_JLCPCB:Q_SOT-23, symbol PCM_JLCPCB-Transistors:PMOS,AO3401A
- added Q16: HL3400, PCM_JLCPCB:Q_SOT-23, symbol PCM_JLCPCB-Transistors:NMOS,HL3400
- added R38, R56, R58, R59, R61, R62, R63, R64, R65, R68: 10K(1%), Capacitor_SMD:C_0603_1608Metric, symbol Device:R
- added R57, R60: 2K2(5%), Capacitor_SMD:C_0603_1608Metric, symbol Device:R
- J1: value CON19x1-LEFT -> CON16x1-LEFT; footprint Connector_PinSocket_2.54mm:PinSocket_1x19_P2.54mm_Vertical -> Connector_PinSocket_2.54mm:PinSocket_1x16_P2.54mm_Vertical; symbol Connector:Conn_01x19_Pin -> Connector:Conn_01x16_Pin
- J10, J9, JP2: now left out of the parts list
- J2: value CON19x1-RIGHT -> CON16x1-RIGHT; footprint Connector_PinSocket_2.54mm:PinSocket_1x19_P2.54mm_Vertical -> Connector_PinSocket_2.54mm:PinSocket_1x16_P2.54mm_Vertical; symbol Connector:Conn_01x19_Pin -> Connector:Conn_01x16_Pin
- J3: FT Position Offset (none) -> 0,2.38; JLCPCB_CORRECTION 0;2.38;0 -> (none)
- J4: value Screw_Terminal_01x10 -> Screw_Terminal_01x09; footprint TerminalBlock_Phoenix:TerminalBlock_Phoenix_MKDS-1,5-10-5.08_1x10_P5.08mm_Horizontal -> TerminalBlock_Phoenix:TerminalBlock_Phoenix_MKDS-1,5-9_1x09_P5.00mm_Horizontal; symbol Connector:Screw_Terminal_01x10 -> Connector:Screw_Terminal_01x09
- Q1, Q2, Q3, Q4, Q5: FT Rotation Offset (none) -> 180
- R10, R12, R13, R15, R5: value 2K(5%) -> 2K2(5%); LCSC C22975 -> C4190
- R17: value 120(1%) -> 120R(1%); LCSC C22975 -> C22787
- R18, R25, R26, R30, R31, R32, R33, R37, R39, R40, R41, R42, R47, R48, R49, R50: value 20K(5%) -> 22K(5%); LCSC C22975 -> C31850
- R19, R21: value 3k -> 2K2(5%); footprint (none) -> Capacitor_SMD:C_0603_1608Metric; LCSC (none) -> C4190
- R20, R22: value 3k -> 10K(1%); footprint (none) -> Capacitor_SMD:C_0603_1608Metric; LCSC (none) -> C25804
- R24, R27, R28, R29, R34, R35, R36, R43, R44, R45, R46, R51, R52, R53, R54, R55: value 2k(5%) -> 2K2(5%); LCSC C22975 -> C4190
- R3: footprint Capacitor_SMD:C_0805_2012Metric -> Capacitor_SMD:C_0603_1608Metric; LCSC C17560 -> C31850
- U1: FT Position Offset (none) -> 0,-2.03; FT Rotation Offset (none) -> -90
- U13, U14, U15, U16, U17, U18, U19, U2, U20, U21, U22, U23, U24, U25, U26, U27, U28: FT Rotation Offset (none) -> -90
- U29, U4, U5: FT Rotation Offset (none) -> 90
- U3: JLCPCB_CORRECTION 0;0;180 -> (none)
Connections:
- net Dust sensor loop 1 is gone; now on net GND: U10. (Output)
- net High pressure signal is gone; now on net High pressure signal (24V): K1.14
- net VDD33 is gone; now on net 3.3V: C1.2, C2.2, C3.1, C5.1, C8.1, J1.1 (Pin_1), R5.1, R9.1, U1.2 (3V3), U2.6 (VDD), U2.7 (VREGIN), U3.2 (VO)
- net 24V: now also C10.1, C11.1, J4.8 (Pin_8), R20.2, U4.1 (VIN), J11.3 (Pin_3), J5.3 (Pin_3), J7.1 (Pin_1), J7.2 (Pin_2), J7.3 (Pin_3), J7.4 (Pin_4), J7.5 (Pin_5), J7.6 (Pin_6), J7.7 (Pin_7), J7.8 (Pin_8), Q12.2 (S), Q14.2 (S), Q8.2 (S), Q9.2 (S), R56.2, R59.2, R62.2
- net 3.3V: now also C13.1, C14.1, J6.3 (Pin_3)
- net GND: now also D1.1, D7.1, J4.9 (Pin_9), BZ1.2 (-), C13.2, C14.2, D13.1, D30.1, D32.1, D33.1, D5.1, J5.1 (Pin_1), J6.1 (Pin_1), J8.1 (Pin_1), Q10.2 (E), Q11.2 (E), Q13.2 (E), Q16.2 (S), Q7.2 (E), R63.2, R64.2, R65.2; no longer J4.7 (Pin_7), J4.8 (Pin_8)
- net IO0: now also U5.11 (A)
- net IO12: now also R19.2, R38.1
- net IO14: now also R57.2, R58.1
- net IO16: now also U5.9 (C)
- net IO17: now also U5.3 (COM_OUT/IN)
- net IO18: now also U29.10 (B)
- net IO19: now also U29.9 (C)
- net IO2: now also R60.2, R61.1
- net IO21: now also U29.3 (COM_OUT/IN)
- net IO23: no longer R16.1, U11.2 (DQ)
- net IO25: now also Q5.1 (G), R15.1, R65.1; no longer Q4.1 (G), R13.1, U29.9 (C), U5.9 (C)
- net IO26: now also Q4.1 (G), R13.1, R64.1; no longer Q2.1 (G), R12.1, U29.10 (B), U5.10 (B)
- net IO27: now also Q2.1 (G), R12.1, R63.1; no longer U29.11 (A), U5.11 (A)
- net IO32: now also R16.1, U11.2 (DQ), J6.2 (Pin_2)
- net IO33: now also Q16.1 (G); no longer Q5.1 (G), R15.1, U29.3 (COM_OUT/IN), U5.3 (COM_OUT/IN)
- net IO4: now also U5.10 (B)
- net IO5: now also U29.11 (A)
- net Main power relay (+): no longer D12.2 (A)
- net at R22.2: now also Q10.1 (B)
- net at J10.1 (Pin_1): now also U24.1; no longer U14.1
- net at J10.10 (Pin_10): now also U15.1; no longer U22.1
- net at J10.11 (Pin_11): now also U13.1; no longer U23.1
- net at J10.12 (Pin_12): now also U14.1; no longer U24.1
- net at J10.2 (Pin_2): now also U23.1; no longer U13.1
- net at J10.3 (Pin_3): now also U22.1; no longer U15.1
- net at J10.4 (Pin_4): now also U21.1; no longer U16.1
- net at J10.5 (Pin_5): now also U20.1; no longer U17.1
- net at J10.6 (Pin_6): now also U19.1; no longer U18.1
- net at J10.7 (Pin_7): now also U18.1; no longer U19.1
- net at J10.8 (Pin_8): now also U17.1; no longer U20.1
- net at J10.9 (Pin_9): now also U16.1; no longer U21.1
- net at R15.2: now also D13.2; no longer D7.2
- net at U28.1: now also J9.1 (Pin_1); no longer J9.4 (Pin_4)
- net at U25.1: now also J9.4 (Pin_4); no longer J9.1 (Pin_1)
- net High pressure signal (24V): now reaches J9.3 (Pin_3)
- net High pressure signal (24V): now also U26.1, J11.1 (Pin_1); no longer U27.1
- net IO13: now reaches R21.2
- net IO13: now also J1.15 (Pin_15), R22.1, U1.16 (MTCK/GPIO13/ADC2_CH4)
- net 5V: now reaches J1.16 (Pin_16)
- net 5V: now also C6.1, D6.1, JP2.2 (B), R10.1, U3.3 (VI), J8.3 (Pin_3), R68.2
- net Low pressure signal (24V): now reaches J9.2 (Pin_2)
- net Low pressure signal (24V): now also K1.12, U27.1, J11.2 (Pin_2); no longer U26.1
- net at R13.2: now also D5.2
- removed net 24V_IN: C10.1, C11.1, J4.1 (Pin_1), J4.3 (Pin_3), J4.5 (Pin_5), J4.9 (Pin_9), U4.1 (VIN)
- removed net Dust sensor loop 2: J1.15 (Pin_15), R17.2, U1.16 (MTCK/GPIO13/ADC2_CH4)
- net Dust warning signal 1: no longer names the net of R20.1
- net Dust warning signal 1: now also Q10.3 (C), Q9.1 (G); no longer D11.2 (A)
- net Dust warning signal 2: no longer names the net of R21.1
- net Dust warning signal 2: now also D7.2; no longer D10.2 (A)
- removed net EXT_5V: C6.1, D6.1, J1.19 (Pin_19), J4.10 (Pin_10), JP2.2 (B), R10.1, U3.3 (VI)
- net IO34 renamed Dust sensor loop
- net Dust sensor loop: now also R17.2, U10. (Output), J5.2 (Pin_2)
- net LEDStrip1(-) renamed Dimmer2(-)
- net Dimmer2(-): now also Q4.3 (D); no longer Q5.3 (D)
- net LEDStrip2(-) renamed Switch24V_R
- net Switch24V_R: now also D10.2 (A), Q9.3 (D); no longer Q4.3 (D)
- net LEDStrip3(-) renamed Dimmer1(-)
- net Dimmer1(-): now also J4.3 (Pin_3), K2.A1; no longer J4.6 (Pin_6)
- net Low pressure signal: no longer names the net of R19.1
- net Low pressure signal: now also D33.2; no longer K1.12
- removed net Main power relay (-): K2.A1, R22.1
- new net: Q13.1 (B), R61.2
- new net: Q11.1 (B), R58.2
- new net: Q7.1 (B), R38.2
- new net: Q7.3 (C), Q8.1 (G), R56.1
- new net: Q11.3 (C), Q12.1 (G), R59.1
- new net: D32.2, R60.1
- new net: Q13.3 (C), Q14.1 (G), R62.1
- new net: D30.2, R57.1
- new net AddressableLED: J8.2 (Pin_2), Q16.3 (D), R68.1
- new net Dimmer3(-): J4.1 (Pin_1), Q5.3 (D)
- new net Switch24V_G: D12.2 (A), J4.6 (Pin_6), Q12.3 (D)
- new net Switch24V_Y: D11.2 (A), J4.5 (Pin_5), Q8.3 (D)
- new net Switch24V_Z: BZ1.1 (+), J4.7 (Pin_7), Q14.3 (D)
- no-connect marks 26 -> 18
Other:
- note added: "GPIO0 is strapping pin for ESP32, must be be input only"
- note added: "GPIO2 is strapping pin for ESP32, must be be input only"
- note added: "GPIO5 is strapping pin for ESP32, must be be input only"
- note added: "LED Controllers"
- note removed: "Flashing warning light"
- note removed: "Input potentiometer"
- note removed: "ON = Dust < ~90%"
- note removed: "ON = Dust > ~80%"
- note removed: "ON = Dust > ~90%"
- note removed: "Optocoupler Module"
- note removed: "Pulldown (for unpowered MCU)"
- note removed: "Scale module"
- moved on the sheet: D10, D11, D12, J9, R16, R17, U29

Commit message: Organize schematic
Other:
- note added: "Multiplexers"
- note added: "Optocoupler inputs"
- note added: "Switches 24V"
- note added: "Switches 5V"
- note added: "Switches GND"
- note removed: "ESP32 Controller board"
- note removed: "LED Controllers"
- note removed: "LED Strip Dimmers"
- moved on the sheet: BZ1, C1, C10, C11, C12, C13, C14, C2, C3, C4, C5, C6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

Commit message: Add ESD protection and other safety improvements
Parts:
- removed C13, C14, C2, C4, C5: 0.1uF/50V(10%), Capacitor_SMD:C_0402_1005Metric, symbol Device:C
- removed J4: Screw_Terminal_01x09, TerminalBlock_Phoenix:TerminalBlock_Phoenix_MKDS-1,5-9_1x09_P5.00mm_Horizontal, symbol Connector:Screw_Terminal_01x09
- removed Q11, Q13, Q7: MMBT3904 100-300, PCM_JLCPCB:Q_SOT-23, symbol PCM_JLCPCB-Transistors:NPN,MMBT3904 100-300
- removed Q12, Q14, Q8: AO3401A, PCM_JLCPCB:Q_SOT-23, symbol PCM_JLCPCB-Transistors:PMOS,AO3401A
- removed Q16: HL3400, PCM_JLCPCB:Q_SOT-23, symbol PCM_JLCPCB-Transistors:NMOS,HL3400
- removed R16: 5K1(1%), Resistor_SMD:R_0402_1005Metric, symbol Device:R
- removed R17: 120R(1%), Capacitor_SMD:C_0603_1608Metric, symbol Device:R
- removed R19, R21, R24, R27, R28, R29, R34, R35, R36, R43, R44, R45, R46, R51, R52, R53, R54, R55, R57, R60: 2K2(5%), Capacitor_SMD:C_0603_1608Metric, symbol Device:R
- removed R20, R22, R38, R56, R58, R59, R61, R62, R68: 10K(1%), Capacitor_SMD:C_0603_1608Metric, symbol Device:R
- added C13, C14, C15, C16, C17, C2, C4, C5: 100nF, PCM_JLCPCB:C_0603, symbol PCM_JLCPCB-Capacitors:0603,100nF
- added C18, C19, C20, C22: 1uF, PCM_JLCPCB:C_0603, symbol PCM_JLCPCB-Capacitors:0603,1uF
- added D31, D36: 1N5819WS, PCM_JLCPCB:D_SOD-323, symbol PCM_JLCPCB-Diodes:Schottky,1N5819WS
- added D34, D35: SMF26A, PCM_JLCPCB:D_SOD-123FL, symbol PCM_JLCPCB-Diodes:TVS-Uni,SMF26A
- added D38: TT0421SAX, PCM_JLCPCB:D_DFN0603-2L, symbol PCM_JLCPCB-Diodes:TVS-Bi,H3V3L10B
- added D39: BZT52B3V3, PCM_JLCPCB:D_SOD-123, symbol PCM_JLCPCB-Diodes:Zener,BZT52B3V3
- added J12: Screw_Terminal_01x10, TerminalBlock_Phoenix:TerminalBlock_Phoenix_MKDS-1,5-10_1x10_P5.00mm_Horizontal, symbol Connector:Screw_Terminal_01x10
- added Q15, Q18, Q20: AO3401A, PCM_JLCPCB:Q_SOT-23, symbol PCM_JLCPCB-Transistors:PMOS,AO3401A
- added Q17, Q19, Q6: MMBT3904 100-300, PCM_JLCPCB:Q_SOT-23, symbol PCM_JLCPCB-Transistors:NPN,MMBT3904 100-300
- added R16: 100Ω, PCM_JLCPCB:R_0402, symbol PCM_JLCPCB-Resistors:0402,100Ω
- added R17, R20, R71, R73, R75, R77, R79, R81: 10kΩ, PCM_JLCPCB:R_0603, symbol PCM_JLCPCB-Resistors:0603,10kΩ
- added R21, R72, R76, R80: 15kΩ, PCM_JLCPCB:R_0603, symbol PCM_JLCPCB-Resistors:0603,15kΩ
- added R22, R70, R74, R78: 2.2kΩ, PCM_JLCPCB:R_0603, symbol PCM_JLCPCB-Resistors:0603,2.2kΩ
- added R23, R69: 300Ω, PCM_JLCPCB:R_1206, symbol PCM_JLCPCB-Resistors:1206,300Ω
- added R24, R27, R28, R29, R34, R35, R36, R43, R44, R45, R46, R51, R52, R53, R54, R55: 4.7kΩ, PCM_JLCPCB:R_0603, symbol PCM_JLCPCB-Resistors:0603,4.7kΩ
- added R66: 120Ω, PCM_JLCPCB:R_0603, symbol PCM_JLCPCB-Resistors:0603,120Ω
- added R67: 3.3kΩ, PCM_JLCPCB:R_0402, symbol PCM_JLCPCB-Resistors:0402,3.3kΩ
- added U6: SN74LVC1T45DBVR, Package_TO_SOT_SMD:SOT-23-6, symbol Logic_LevelTranslator:SN74LVC1T45DBV
- S1: now not fitted; now left out of the parts list
Connections:
- net 24V: now also C18.1, C19.1, C20.1, C22.1, D31.1, D36.1, J12.8 (Pin_8), Q15.2 (S), Q18.2 (S), Q20.2 (S), R17.1, R73.1, R77.1, R81.1; no longer V1.1
- net 3.3V: now also C13.1, C14.1, C17.1, C2.2, C5.1, R67.1, U6.1 (VCCA), U6.5 (DIR)
- net 5V: now also C16.1, U6.6 (VCCB)
- net AddressableLED: now also U6.4 (B)
- net Dimmer1(-): now also D36.2, J12.7 (Pin_7)
- net Dimmer2(-): now also J12.6 (Pin_6)
- net Dimmer3(-): now also J12.5 (Pin_5)
- net Dust sensor loop: now also D35.1, R23.1; no longer J1.5 (Pin_5), U1.6 (GPIO34/ADC1_CH6)
- net EN: now also C4.1
- net GND: now also C13.2, C14.2, C15.2, C16.2, C17.2, C18.2, C19.2, C2.1, C20.2, C22.2, C4.2, C5.2, D34.2, D35.2, D38.1, D39.2, J12.10 (Pin_10), Q17.2 (E), Q19.2 (E), Q6.2 (E), R24.2, R27.2, R28.2, R29.2, R34.2, R35.2, R36.2, R43.2, R44.2, R45.2, R46.2, R51.2, R52.2, R53.2, R54.2, R55.2, R66.2, U6.2 (GND)
- net IO12: now also R70.2, R71.2
- net IO13: now also R20.2, R22.2
- net IO14: now also R74.2, R75.2
- net IO2: now also R78.2, R79.2
- net IO32: now also R16.2, R67.2; no longer J6.2 (Pin_2), U11.2 (DQ)
- net IO33: now also U6.3 (A)
- net Switch24V_G: now also J12.3 (Pin_3), Q18.3 (D)
- net Switch24V_R: now also J12.1 (Pin_1)
- net Switch24V_Y: now also J12.2 (Pin_2), Q15.3 (D)
- net Switch24V_Z: now also J12.4 (Pin_4), Q20.3 (D)
- net at D33.2: now also R70.1
- net at Q9.1 (G): now also R17.2, R21.2; no longer Q10.3 (C)
- net at D28.1: now also R53.1
- net at D17.1: now also R28.1
- net at D18.1: now also R34.1
- net at Q10.1 (B): now also R20.1
- net at D26.1: now also R51.1
- net at D14.1: now also R29.1
- net at D21.1: now also R55.1
- net at D23.1: now also R44.1
- net at D19.1: now also R35.1
- net at D27.1: now also R52.1
- net at D25.1: now also R46.1
- net at D32.2: now also R78.1
- net at D22.1: now also R43.1
- net at D16.1: now also R27.1
- net at D24.1: now also R45.1
- net at D7.2: now also R22.1
- net at D20.1: now also R36.1
- net at D15.1: now also R24.1
- net at D30.2: now also R74.1
- net at D29.1: now also R54.1
- new net: Q19.1 (B), R79.1
- new net: Q10.3 (C), R21.1
- new net: Q19.3 (C), R80.1
- new net: Q17.1 (B), R75.1
- new net: Q17.3 (C), R76.1
- new net: Q6.1 (B), R71.1
- new net: Q15.1 (G), R72.2, R73.2
- new net: Q6.3 (C), R72.1
- new net: R23.2, R69.1
- new net: Q20.1 (G), R80.2, R81.2
- new net: Q18.1 (G), R76.2, R77.2
- new net 24V_RAW: D31.2, D34.1, J12.9 (Pin_9), V1.1
- new net IO34: C15.1, D39.1, J1.5 (Pin_5), R66.1, R69.2, U1.6 (GPIO34/ADC1_CH6)
- new net Onewire bus: D38.2, J6.2 (Pin_2), R16.1, U11.2 (DQ)
Other:
- note added: "Flyback"
- moved on the sheet: D30, D32, D33, D7, J11, J8

Commit message: Final tweaks. Ordered from JLCPCB
Parts:
- removed C11: 0.1uF/50V(10%), Capacitor_SMD:C_0402_1005Metric, symbol Device:C
- added C11: 100nF, PCM_JLCPCB:C_0603, symbol PCM_JLCPCB-Capacitors:0603,100nF
- C10, C12: footprint Capacitor_THT:CP_Radial_D6.3mm_P2.50mm -> Capacitor_THT:CP_Radial_D10.0mm_P5.00mm
- J12: now left out of the parts list
- R1, R2, R63, R64, R65, R9: value 10K(1%) -> 10kΩ; footprint Capacitor_SMD:C_0603_1608Metric -> PCM_JLCPCB:R_0603
- R10, R12, R13, R15, R5: value 2K2(5%) -> 2.2kΩ; footprint Capacitor_SMD:C_0603_1608Metric -> PCM_JLCPCB:R_0603
- R18, R25, R26, R3, R30, R31, R32, R33, R37, R39, R4, R40, R41, R42, R47, R48, R49, R50: footprint Capacitor_SMD:C_0603_1608Metric -> PCM_JLCPCB:R_0603
Connections:
- net 24V: now also C11.2
- net GND: now also C11.1
- net Switch24V: now reaches D8.1, L1.1, U4.2 (OUTPUT)
